File: SENSOR_HARDWARE/$SENSOR_HARDWARE.sch (KiCad schematic (older format))
At the start: 27 parts, among them IC1 ATTINY85-S, P1 CONN_02X03, P2 NRF24L01+, T1 LM335, U1 LM358

Commit message: created SOD-123 footprint
finished assigning all footprints. yipee
Parts:
- F1: footprint (none) -> Resistors_SMD:R_0603_HandSoldering
Changed lines of the file:
@@
 F 0 "F1" H 3650 1700 40  0000 C CNN
 F 1 "500mA" H 3450 1600 40  0000 C CNN
-F 2 "" H 3550 1650 60  0001 C CNN
+F 2 "Resistors_SMD:R_0603_HandSoldering" H 3550 1650 60  0001 C CNN
 F 3 "" H 3550 1650 60  0000 C CNN
 	1    3550 1650
